File: scale-infrared-digitiser.kicad_sch (KiCad schematic)
At the start: 0 parts

Commit message: schematic design completed
Parts:
- added C1, C10, C11, C12, C15, C16, C17, C18, C21, C22, C23, C24, C3, C4, C5, C9: 5.1p, Capacitor_SMD:C_0603_1608Metric, symbol Device:C_Small
- added C13, C14, C19, C2, C20, C25, C6, C7, C8: 1u, Capacitor_SMD:C_0603_1608Metric, symbol Device:C_Small
- added D_photo0, D_photo1, D_photo10, D_photo11, D_photo12, D_photo13, D_photo14, D_photo15, D_photo2, D_photo3, D_photo4, D_photo5, D_photo6, D_photo7, D_photo8, D_photo9: VEMD10940FX01, Samacsys:VEMD10940FX01, symbol Samacsys:VEMD10940FX01
- added IC0, IC1, IC2, IC3: LM324PT, Samacsys:SOP65P640X120-14N, symbol Samacsys:LM324PT
- added IC4, IC5: 74HC4067PW,118, Samacsys:SOP65P640X110-24N, symbol Samacsys:74HC4067PW,118
- added J0: Conn_02x04_TRNS, Connector_PinHeader_2.54mm:PinHeader_2x04_P2.54mm_Vertical, symbol Connector_Generic:Conn_02x04_Top_Bottom
- added J1: Conn_02x04_RECV, Connector_PinHeader_2.54mm:PinHeader_2x04_P2.54mm_Vertical, symbol Connector_Generic:Conn_02x04_Top_Bottom
- added LED0, LED1, LED10, LED11, LED12, LED13, LED14, LED15, LED2, LED3, LED4, LED5, LED6, LED7, LED8, LED9: VSMB10940, Samacsys:VSMB10940, symbol Samacsys:VSMB10940
- added Q1, Q10, Q11, Q12, Q13, Q14, Q15, Q16, Q2, Q3, Q4, Q5, Q6, Q7, Q8, Q9: T2N7002AK, Package_TO_SOT_SMD:SOT-23, symbol Transistor_FET:T2N7002AK
- added R1, R10, R11, R12, R13, R14, R15, R16, R2, R3, R4, R5, R6, R7, R8, R9: 200R, Resistor_SMD:R_0603_1608Metric, symbol Device:R_Small
- added R17, R20, R21, R22, R23, R24, R25, R26, R27, R28, R29, R30, R31, R32, R33, R34: 750k, Resistor_SMD:R_0603_1608Metric, symbol Device:R_Small
- added R18: 115k, Resistor_SMD:R_0603_1608Metric, symbol Device:R_Small
- added R19: 3.57k, Resistor_SMD:R_0603_1608Metric, symbol Device:R_Small
Connections:
- new net: LED10.1 (K), Q11.3 (D)
- new net: LED10.2 (A), R11.1
- new net: LED11.2 (A), R12.1
- new net: LED9.1 (K), Q10.3 (D)
- new net: LED9.2 (A), R10.1
- new net: LED14.2 (A), R15.1
- new net: C3.1, IC2.14 (OUTPUT_4), R20.2
- new net: LED8.1 (K), Q9.3 (D)
- new net: LED8.2 (A), R9.1
- new net: LED2.1 (K), Q3.3 (D)
- new net: C17.2, IC1.8 (OUTPUT_3), R29.1
- new net: LED4.1 (K), Q5.3 (D)
- new net: LED4.2 (A), R5.1
- new net: C15.2, IC1.1 (OUTPUT_1), R27.1
- new net: C4.1, IC2.7 (OUTPUT_2), R21.2
- new net: C18.1, IC1.14 (OUTPUT_4), R30.2
- new net: C16.1, IC1.7 (OUTPUT_2), R28.2
- new net: LED6.1 (K), Q7.3 (D)
- new net: C11.2, IC0.8 (OUTPUT_3), R25.1
- new net: LED2.2 (A), R3.1
- new net: LED13.1 (K), Q14.3 (D)
- new net: LED5.2 (A), R6.1
- new net: C9.2, IC0.1 (OUTPUT_1), R23.1
- new net: LED7.1 (K), Q8.3 (D)
- new net: LED7.2 (A), R8.1
- new net: LED11.1 (K), Q12.3 (D)
- new net: C12.1, IC0.14 (OUTPUT_4), R26.2
- new net: LED0.2 (A), R1.1
- new net: C23.2, IC3.8 (OUTPUT_3), R33.1
- new net: LED12.1 (K), Q13.3 (D)
- new net: LED6.2 (A), R7.1
- new net: LED14.1 (K), Q15.3 (D)
- new net: C5.2, IC2.8 (OUTPUT_3), R22.1
- new net: C22.1, IC3.7 (OUTPUT_2), R32.2
- new net: LED3.2 (A), R4.1
- new net: LED3.1 (K), Q4.3 (D)
- new net: LED5.1 (K), Q6.3 (D)
- new net: C21.2, IC3.1 (OUTPUT_1), R31.1
- new net: C1.2, IC2.1 (OUTPUT_1), R17.1
- new net: LED12.2 (A), R13.1
- new net: LED0.1 (K), Q1.3 (D)
- new net: LED1.2 (A), R2.1
- new net: C10.1, IC0.7 (OUTPUT_2), R24.2
- new net: C24.1, IC3.14 (OUTPUT_4), R34.2
- new net: LED1.1 (K), Q2.3 (D)
- new net: LED13.2 (A), R14.1
- new net: LED15.1 (K), Q16.3 (D)
- new net: LED15.2 (A), R16.1
- new net 3V3: IC0.4 (VCC+), IC1.4 (VCC+), IC2.4 (VCC+), IC3.4 (VCC+), IC4.24 (VCC), IC5.24 (VCC), J0.5 (Pin_5), J1.5 (Pin_5), R1.2, R10.2, R11.2, R12.2, R13.2, R14.2, R15.2, R16.2, R18.2, R2.2, R3.2, R4.2, R5.2, R6.2, R7.2, R8.2, R9.2
- new net GND: C13.2, C14.2, C19.2, C2.2, C20.2, C25.2, C6.2, C7.1, C8.2, D_photo0.2 (A), D_photo1.2 (A), D_photo10.2 (A), D_photo11.2 (A), D_photo12.2 (A), D_photo13.2 (A), D_photo14.2 (A), D_photo15.2 (A), D_photo2.2 (A), D_photo3.2 (A), D_photo4.2 (A), D_photo5.2 (A), D_photo6.2 (A), D_photo7.2 (A), D_photo8.2 (A), D_photo9.2 (A), IC0.11 (VCC-), IC1.11 (VCC-), IC2.11 (VCC-), IC3.11 (VCC-), IC4.12 (GND), IC4.15 (~{E}), IC5.12 (GND), IC5.15 (~{E}), J0.7 (Pin_7), J0.8 (Pin_8), J1.7 (Pin_7), J1.8 (Pin_8), Q1.2 (S), Q10.2 (S), Q11.2 (S), Q12.2 (S), Q13.2 (S), Q14.2 (S), Q15.2 (S), Q16.2 (S), Q2.2 (S), Q3.2 (S), Q4.2 (S), Q5.2 (S), Q6.2 (S), Q7.2 (S), Q8.2 (S), Q9.2 (S), R19.1
- new net LED_CTL_0: IC4.9 (Y0), Q1.1 (G)
- new net LED_CTL_1: IC4.8 (Y1), Q2.1 (G)
- new net LED_CTL_10: IC4.21 (Y10), Q11.1 (G)
- new net LED_CTL_11: IC4.20 (Y11), Q12.1 (G)
- new net LED_CTL_12: IC4.19 (Y12), Q13.1 (G)
- new net LED_CTL_13: IC4.18 (Y13), Q14.1 (G)
- new net LED_CTL_14: IC4.17 (Y14), Q15.1 (G)
- new net LED_CTL_15: IC4.16 (Y15), Q16.1 (G)
- new net LED_CTL_2: IC4.7 (Y2), Q3.1 (G)
- new net LED_CTL_3: IC4.6 (Y3), Q4.1 (G)
- new net LED_CTL_4: IC4.5 (Y4), Q5.1 (G)
- new net LED_CTL_5: IC4.4 (Y5), Q6.1 (G)
- new net LED_CTL_6: IC4.3 (Y6), Q7.1 (G)
- new net LED_CTL_7: IC4.2 (Y7), Q8.1 (G)
- new net LED_CTL_8: IC4.23 (Y8), Q9.1 (G)
- new net LED_CTL_9: IC4.22 (Y9), Q10.1 (G)
- new net MCU_RECV_DAT: IC5.1 (Z), J1.6 (Pin_6)
- new net MCU_TRNS_CTL: IC4.1 (Z), J0.6 (Pin_6)
- new net NON_INVERTING_REF: C13.1, C14.1, C19.1, C2.1, C20.1, C25.1, C6.1, C7.2, C8.1, IC0.10 (NON-INVERTING_INPUT_3), IC0.12 (NON-INVERTING_INPUT_4), IC0.3 (NON-INVERTING_INPUT_1), IC0.5 (NON-INVERTING_INPUT_2), IC1.10 (NON-INVERTING_INPUT_3), IC1.12 (NON-INVERTING_INPUT_4), IC1.3 (NON-INVERTING_INPUT_1), IC1.5 (NON-INVERTING_INPUT_2), IC2.10 (NON-INVERTING_INPUT_3), IC2.12 (NON-INVERTING_INPUT_4), IC2.3 (NON-INVERTING_INPUT_1), IC2.5 (NON-INVERTING_INPUT_2), IC3.10 (NON-INVERTING_INPUT_3), IC3.12 (NON-INVERTING_INPUT_4), IC3.3 (NON-INVERTING_INPUT_1), IC3.5 (NON-INVERTING_INPUT_2), R18.1, R19.2
- new net PHT_DAT_0: C9.1, D_photo0.1 (K), IC0.2 (INVERTING_INPUT_1), IC5.9 (Y0), R23.2
- new net PHT_DAT_1: C10.2, D_photo1.1 (K), IC0.6 (INVERTING_INPUT_2), IC5.8 (Y1), R24.1
- new net PHT_DAT_10: C23.1, D_photo10.1 (K), IC3.9 (INVERTING_INPUT_3), IC5.21 (Y10), R33.2
- new net PHT_DAT_11: C24.2, D_photo11.1 (K), IC3.13 (INVERTING_INPUT_4), IC5.20 (Y11), R34.1
- new net PHT_DAT_12: C1.1, D_photo12.1 (K), IC2.2 (INVERTING_INPUT_1), IC5.19 (Y12), R17.2
- new net PHT_DAT_13: C4.2, D_photo13.1 (K), IC2.6 (INVERTING_INPUT_2), IC5.18 (Y13), R21.1
- new net PHT_DAT_14: C5.1, D_photo14.1 (K), IC2.9 (INVERTING_INPUT_3), IC5.17 (Y14), R22.2
- new net PHT_DAT_15: C3.2, D_photo15.1 (K), IC2.13 (INVERTING_INPUT_4), IC5.16 (Y15), R20.1
- new net PHT_DAT_2: C11.1, D_photo2.1 (K), IC0.9 (INVERTING_INPUT_3), IC5.7 (Y2), R25.2
- new net PHT_DAT_3: C12.2, D_photo3.1 (K), IC0.13 (INVERTING_INPUT_4), IC5.6 (Y3), R26.1
- new net PHT_DAT_4: C15.1, D_photo4.1 (K), IC1.2 (INVERTING_INPUT_1), IC5.5 (Y4), R27.2
- new net PHT_DAT_5: C16.2, D_photo5.1 (K), IC1.6 (INVERTING_INPUT_2), IC5.4 (Y5), R28.1
- new net PHT_DAT_6: C17.1, D_photo6.1 (K), IC1.9 (INVERTING_INPUT_3), IC5.3 (Y6), R29.2
- new net PHT_DAT_7: C18.2, D_photo7.1 (K), IC1.13 (INVERTING_INPUT_4), IC5.2 (Y7), R30.1
- new net PHT_DAT_8: C21.1, D_photo8.1 (K), IC3.2 (INVERTING_INPUT_1), IC5.23 (Y8), R31.2
- new net PHT_DAT_9: C22.2, D_photo9.1 (K), IC3.6 (INVERTING_INPUT_2), IC5.22 (Y9), R32.1
- new net SEL_RECV_0: IC5.10 (S0), J1.4 (Pin_4)
- new net SEL_RECV_1: IC5.11 (S1), J1.3 (Pin_3)
- new net SEL_RECV_2: IC5.14 (S2), J1.2 (Pin_2)
- new net SEL_RECV_3: IC5.13 (S3), J1.1 (Pin_1)
- new net SEL_TRNS_0: IC4.10 (S0), J0.4 (Pin_4)
- new net SEL_TRNS_1: IC4.11 (S1), J0.3 (Pin_3)
- new net SEL_TRNS_2: IC4.14 (S2), J0.2 (Pin_2)
- new net SEL_TRNS_3: IC4.13 (S3), J0.1 (Pin_1)
- no-connect marks 0 -> 32
Other:
- note added: "Inputs and Outputs"
- note added: "Receiver array"
- note added: "Transmitter array"
