File: scale-infrared-digitiser.kicad_sch (KiCad schematic)
At the start: 111 parts, among them IC0 LM324PT, IC1 LM324PT, IC2 LM324PT, IC3 LM324PT, IC4 74HC4067PW,118, IC5 74HC4067PW,118, J0 Conn_02x04_TRNS, J1 Conn_02x04_RECV, Q1 T2N7002AK, Q10 T2N7002AK, Q11 T2N7002AK, Q12 T2N7002AK, Q13 T2N7002AK, Q14 T2N7002AK, Q15 T2N7002AK, Q16 T2N7002AK, Q2 T2N7002AK, Q3 T2N7002AK, Q4 T2N7002AK, Q5 T2N7002AK, Q6 T2N7002AK, Q7 T2N7002AK, Q8 T2N7002AK, Q9 T2N7002AK

Commit message: laptop work
Connections:
- net 3V3_TRNS: now also J0.6 (Pin_6); no longer J0.5 (Pin_5)
- net LED_CTL_0: now also IC4.8 (Y1); no longer IC4.9 (Y0)
- net LED_CTL_1: now also IC4.7 (Y2); no longer IC4.8 (Y1)
- net LED_CTL_2: now also IC4.6 (Y3); no longer IC4.7 (Y2)
- net LED_CTL_3: now also IC4.5 (Y4); no longer IC4.6 (Y3)
- net LED_CTL_4: now also IC4.4 (Y5); no longer IC4.5 (Y4)
- net LED_CTL_5: now also IC4.3 (Y6); no longer IC4.4 (Y5)
- net LED_CTL_6: now also IC4.2 (Y7); no longer IC4.3 (Y6)
- net LED_CTL_7: now also IC4.1 (Z); no longer IC4.2 (Y7)
- net MCU_TRNS_CTL: now also IC4.9 (Y0), J0.5 (Pin_5); no longer IC4.1 (Z), J0.6 (Pin_6)
- net SEL_TRNS_0: now also IC4.13 (S3); no longer IC4.10 (S0)
- net SEL_TRNS_3: now also IC4.10 (S0); no longer IC4.13 (S3)
Changed lines of the file:
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@@
 	(wire
 		(pts
-			(xy 149.86 76.2) (xy 133.35 76.2)
+			(xy 153.67 76.2) (xy 133.35 76.2)
 		)
 		(stroke
@@
 	(wire
 		(pts
-			(xy 149.86 77.47) (xy 149.86 76.2)
+			(xy 153.67 77.47) (xy 153.67 76.2)
 		)
 		(stroke
@@
 	)
 	(label "LED_CTL_7"
-		(at 135.89 101.6 0)
+		(at 135.89 104.14 0)
 		(effects
 			(font
@@
 	)
 	(label "LED_CTL_3"
-		(at 135.89 91.44 0)
+		(at 135.89 93.98 0)
 		(effects
 			(font
@@
 	)
 	(label "LED_CTL_5"
-		(at 135.89 96.52 0)
+		(at 135.89 99.06 0)
 		(effects
 			(font
@@
 	)
 	(label "LED_CTL_0"
-		(at 135.89 83.82 0)
+		(at 135.89 86.36 0)
 		(effects
 			(font
@@
 	)
 	(label "LED_CTL_2"
-		(at 135.89 88.9 0)
+		(at 135.89 91.44 0)
 		(effects
 			(font
@@
 	)
 	(label "MCU_TRNS_CTL"
-		(at 135.89 104.14 0)
+		(at 135.89 83.82 0)
 		(effects
 			(font
@@
 	)
 	(label "LED_CTL_4"
-		(at 135.89 93.98 0)
+		(at 135.89 96.52 0)
 		(effects
 			(font
@@
 	)
 	(label "3V3_TRNS"
-		(at 354.33 43.18 0)
+		(at 354.33 45.72 0)
 		(effects
 			(font
@@
 	)
 	(label "MCU_TRNS_CTL"
-		(at 354.33 45.72 0)
+		(at 354.33 43.18 0)
 		(effects
 			(font
@@
 	)
 	(label "SEL_TRNS_3"
-		(at 105.41 76.2 180)
+		(at 135.89 81.28 0)
 		(effects
 			(font
 				(size 1.27 1.27)
 			)
-			(justify right bottom)
+			(justify left bottom)
 		)
 	)
@@
 	)
 	(label "SEL_TRNS_0"
-		(at 135.89 81.28 0)
+		(at 105.41 76.2 180)
 		(effects
 			(font
 				(size 1.27 1.27)
 			)
-			(justify left bottom)
+			(justify right bottom)
 		)
 	)
@@
 	)
 	(label "LED_CTL_1"
-		(at 135.89 86.36 0)
+		(at 135.89 88.9 0)
 		(effects
 			(font
@@
 	)
 	(label "LED_CTL_6"
-		(at 135.89 99.06 0)
+		(at 135.89 101.6 0)
 		(effects
 			(font
@@
 	(symbol
 		(lib_id "power:GND")
-		(at 149.86 77.47 0)
+		(at 153.67 77.47 0)
 		(unit 1)
 		(exclude_from_sim no)
@@
 		(dnp no)
 		(property "Reference" "#PWR02"
-			(at 149.86 83.82 0)
+			(at 153.67 83.82 0)
 			(effects
 				(font
@@
 		)
 		(property "Value" "GND1"
-			(at 149.86 81.788 0)
+			(at 153.67 81.788 0)
 			(effects
 				(font
@@
 		)
 		(property "Footprint" ""
-			(at 149.86 77.47 0)
+			(at 153.67 77.47 0)
 			(effects
 				(font
@@
 		)
 		(property "Datasheet" ""
-			(at 149.86 77.47 0)
+			(at 153.67 77.47 0)
 			(effects
 				(font
@@
 		)
 		(property "Description" "Power symbol creates a global label with name \"GND\" , ground"
-			(at 149.86 77.47 0)
+			(at 153.67 77.47 0)
 			(effects
 				(font

Commit message: completed design ready for review before assembly
Connections:
- net LED_CTL_10: now also IC4.18 (Y13); no longer IC4.21 (Y10)
- net LED_CTL_11: now also IC4.19 (Y12); no longer IC4.20 (Y11)
- net LED_CTL_12: now also IC4.20 (Y11); no longer IC4.19 (Y12)
- net LED_CTL_13: now also IC4.21 (Y10); no longer IC4.18 (Y13)
- net LED_CTL_14: now also IC4.22 (Y9); no longer IC4.17 (Y14)
- net LED_CTL_15: now also IC4.23 (Y8); no longer IC4.16 (Y15)
- net LED_CTL_5: now also IC4.1 (Z); no longer IC4.3 (Y6)
- net LED_CTL_7: now also IC4.3 (Y6); no longer IC4.1 (Z)
- net LED_CTL_8: now also IC4.16 (Y15); no longer IC4.23 (Y8)
- net LED_CTL_9: now also IC4.17 (Y14); no longer IC4.22 (Y9)
Changed lines of the file:
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@@
 	)
 	(label "LED_CTL_7"
-		(at 135.89 104.14 0)
+		(at 135.89 99.06 0)
 		(effects
 			(font
@@
 	)
 	(label "LED_CTL_15"
-		(at 105.41 83.82 180)
+		(at 105.41 101.6 180)
 		(effects
 			(font
@@
 	)
 	(label "LED_CTL_9"
-		(at 105.41 99.06 180)
+		(at 105.41 86.36 180)
 		(effects
 			(font
@@
 	)
 	(label "LED_CTL_5"
-		(at 135.89 99.06 0)
+		(at 135.89 104.14 0)
 		(effects
 			(font
@@
 	)
 	(label "LED_CTL_11"
-		(at 105.41 93.98 180)
+		(at 105.41 91.44 180)
 		(effects
 			(font
@@
 	)
 	(label "LED_CTL_12"
-		(at 105.41 91.44 180)
+		(at 105.41 93.98 180)
 		(effects
 			(font
@@
 	)
 	(label "LED_CTL_14"
-		(at 105.41 86.36 180)
+		(at 105.41 99.06 180)
 		(effects
 			(font
@@
 	)
 	(label "LED_CTL_10"
-		(at 105.41 96.52 180)
+		(at 105.41 88.9 180)
 		(effects
 			(font
@@
 	)
 	(label "LED_CTL_8"
-		(at 105.41 101.6 180)
+		(at 105.41 83.82 180)
 		(effects
 			(font
@@
 	)
 	(label "LED_CTL_13"
-		(at 105.41 88.9 180)
-		(effects
-			(font
+		(at 105.41 96.52 180)
+		(effects
+			(font

Commit message: revised DFM submitted to JLCPCB
Parts:
- renumbered D_photo0 to DPht0, D_photo1 to DPht1, D_photo10 to DPht10, D_photo11 to DPht11, D_photo12 to DPht12, D_photo13 to DPht13, D_photo14 to DPht14, D_photo15 to DPht15, D_photo2 to DPht2, D_photo3 to DPht3, D_photo4 to DPht4, D_photo5 to DPht5, D_photo6 to DPht6, D_photo7 to DPht7, D_photo8 to DPht8, D_photo9 to DPht9
Changed lines of the file:
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@@
 	)
 	(symbol
-		(lib_name "VSMB10940_1")
 		(lib_id "Samacsys:VSMB10940")
 		(at 193.04 39.37 0)
@@
 	)
 	(symbol
-		(lib_name "VEMD10940FX01_1")
 		(lib_id "Samacsys:VEMD10940FX01")
 		(at 297.18 165.1 0)
@@
 		(on_board yes)
 		(dnp no)
-		(property "Reference" "D_photo6"
+		(property "Reference" "DPht6"
 			(at 297.688 160.02 0)
 			(effects
@@
 			(project "scale-infrared-digitiser"
 				(path "/30c568d4-c8fa-43dd-998e-54c85dfa19bf"
-					(reference "D_photo6")
+					(reference "DPht6")
 					(unit 1)
 				)
@@
 	)
 	(symbol
-		(lib_name "VSMB10940_1")
 		(lib_id "Samacsys:VSMB10940")
 		(at 177.8 39.37 0)
@@
 	)
 	(symbol
-		(lib_name "VEMD10940FX01_1")
 		(lib_id "Samacsys:VEMD10940FX01")
 		(at 128.27 224.79 0)
@@
 		(on_board yes)
 		(dnp no)
-		(property "Reference" "D_photo10"
+		(property "Reference" "DPht10"
 			(at 128.778 219.71 0)
 			(effects
@@
 			(project "scale-infrared-digitiser"
 				(path "/30c568d4-c8fa-43dd-998e-54c85dfa19bf"
-					(reference "D_photo10")
+					(reference "DPht10")
 					(unit 1)
 				)
@@
 	)
 	(symbol
-		(lib_name "VEMD10940FX01_1")
 		(lib_id "Samacsys:VEMD10940FX01")
 		(at 256.54 165.1 0)
@@
 		(on_board yes)
 		(dnp no)
-		(property "Reference" "D_photo4"
+		(property "Reference" "DPht4"
 			(at 257.048 160.02 0)
 			(effects
@@
 			(project "scale-infrared-digitiser"
 				(path "/30c568d4-c8fa-43dd-998e-54c85dfa19bf"
-					(reference "D_photo4")
+					(reference "DPht4")
 					(unit 1)
 				)
@@
 	)
 	(symbol
-		(lib_name "VSMB10940_1")
 		(lib_id "Samacsys:VSMB10940")
 		(at 162.56 39.37 0)
@@
 	)
 	(symbol
-		(lib_name "VSMB10940_1")
 		(lib_id "Samacsys:VSMB10940")
 		(at 101.6 39.37 0)
@@
 	)
 	(symbol
-		(lib_name "VEMD10940FX01_1")
 		(lib_id "Samacsys:VEMD10940FX01")
 		(at 297.18 224.79 0)
@@
 		(on_board yes)
 		(dnp no)
-		(property "Reference" "D_photo14"
+		(property "Reference" "DPht14"
 			(at 297.688 219.71 0)
 			(effects
@@
 			(project "scale-infrared-digitiser"
 				(path "/30c568d4-c8fa-43dd-998e-54c85dfa19bf"
-					(reference "D_photo14")
+					(reference "DPht14")
 					(unit 1)
 				)
@@
 	)
 	(symbol
-		(lib_name "VEMD10940FX01_1")
 		(lib_id "Samacsys:VEMD10940FX01")
 		(at 276.86 165.1 0)
@@
 		(on_board yes)
 		(dnp no)
-		(property "Reference" "D_photo7"
+		(property "Reference" "DPht7"
 			(at 277.368 160.02 0)
 			(effects
@@
 			(project "scale-infrared-digitiser"
 				(path "/30c568d4-c8fa-43dd-998e-54c85dfa19bf"
-					(reference "D_photo7")
+					(reference "DPht7")
 					(unit 1)
 				)
@@
 	)
 	(symbol
-		(lib_name "VEMD10940FX01_1")
 		(lib_id "Samacsys:VEMD10940FX01")
 		(at 87.63 165.1 0)
@@
 		(on_board yes)
 		(dnp no)
-		(property "Reference" "D_photo0"
+		(property "Reference" "DPht0"
 			(at 88.138 160.02 0)
 			(effects
@@
 			(project "scale-infrared-digitiser"
 				(path "/30c568d4-c8fa-43dd-998e-54c85dfa19bf"
-					(reference "D_photo0")
+					(reference "DPht0")
 					(unit 1)
 				)
@@
 	)
 	(symbol
-		(lib_name "VSMB10940_1")
 		(lib_id "Samacsys:VSMB10940")
 		(at 147.32 39.37 0)
@@
 	)
 	(symbol
-		(lib_name "VSMB10940_1")
 		(lib_id "Samacsys:VSMB10940")
 		(at 208.28 39.37 0)
@@
 	)
 	(symbol
-		(lib_name "VSMB10940_1")
 		(lib_id "Samacsys:VSMB10940")
 		(at 132.08 39.37 0)
@@
 	)
 	(symbol
-		(lib_name "VSMB10940_1")
 		(lib_id "Samacsys:VSMB10940")
 		(at 254 39.37 0)
@@
 	)
 	(symbol
-		(lib_name "VSMB10940_1")
 		(lib_id "Samacsys:VSMB10940")
 		(at 86.36 39.37 0)
@@
 	)
 	(symbol
-		(lib_name "VSMB10940_1")
 		(lib_id "Samacsys:VSMB10940")
 		(at 71.12 39.37 0)
@@
 	)
 	(symbol
-		(lib_name "VEMD10940FX01_1")
 		(lib_id "Samacsys:VEMD10940FX01")
 		(at 236.22 224.79 0)
@@
 		(on_board yes)
 		(dnp no)
-		(property "Reference" "D_photo13"
+		(property "Reference" "DPht13"
 			(at 236.728 219.71 0)
 			(effects
@@
 			(project "scale-infrared-digitiser"
 				(path "/30c568d4-c8fa-43dd-998e-54c85dfa19bf"
-					(reference "D_photo13")
+					(reference "DPht13")
 					(unit 1)
 				)
@@
 	)
 	(symbol
-		(lib_name "VEMD10940FX01_1")
 		(lib_id "Samacsys:VEMD10940FX01")
 		(at 87.63 224.79 0)
@@
 		(on_board yes)
 		(dnp no)
-		(property "Reference" "D_photo8"
+		(property "Reference" "DPht8"
 			(at 88.138 219.71 0)
 			(effects
@@
 			(project "scale-infrared-digitiser"
 				(path "/30c568d4-c8fa-43dd-998e-54c85dfa19bf"
-					(reference "D_photo8")
+					(reference "DPht8")
 					(unit 1)
 				)
@@
 	)
 	(symbol
-		(lib_name "VEMD10940FX01_1")
 		(lib_id "Samacsys:VEMD10940FX01")
 		(at 276.86 224.79 0)
@@
 		(on_board yes)
 		(dnp no)
-		(property "Reference" "D_photo15"
+		(property "Reference" "DPht15"
 			(at 277.368 219.71 0)
 			(effects
@@
 			(project "scale-infrared-digitiser"
 				(path "/30c568d4-c8fa-43dd-998e-54c85dfa19bf"
-					(reference "D_photo15")
+					(reference "DPht15")
 					(unit 1)
 				)
@@
 	)
 	(symbol
-		(lib_name "VEMD10940FX01_1")
 		(lib_id "Samacsys:VEMD10940FX01")
 		(at 256.54 224.79 0)
@@
 		(on_board yes)
 		(dnp no)
-		(property "Reference" "D_photo12"
+		(property "Reference" "DPht12"
 			(at 257.048 219.71 0)
 			(effects
@@
 			(project "scale-infrared-digitiser"
 				(path "/30c568d4-c8fa-43dd-998e-54c85dfa19bf"
-					(reference "D_photo12")
+					(reference "DPht12")
 					(unit 1)
 				)
@@
 	)
 	(symbol
-		(lib_name "VSMB10940_1")
 		(lib_id "Samacsys:VSMB10940")
 		(at 55.88 39.37 0)
@@
 	)
 	(symbol
-		(lib_name "VSMB10940_1")
 		(lib_id "Samacsys:VSMB10940")
 		(at 223.52 39.37 0)
@@
 	)
 	(symbol
-		(lib_name "VSMB10940_1")
 		(lib_id "Samacsys:VSMB10940")
 		(at 40.64 39.37 0)
@@
 	)
 	(symbol
-		(lib_name "VSMB10940_1")
 		(lib_id "Samacsys:VSMB10940")
 		(at 269.24 39.37 0)
@@
 	)
 	(symbol
-		(lib_name "VSMB10940_1")
 		(lib_id "Samacsys:VSMB10940")
 		(at 238.76 39.37 0)
@@
 	)
 	(symbol
-		(lib_name "VEMD10940FX01_1")
 		(lib_id "Samacsys:VEMD10940FX01")
 		(at 107.95 165.1 0)
@@
 		(on_board yes)
 		(dnp no)
-		(property "Reference" "D_photo3"
+		(property "Reference" "DPht3"
 			(at 108.458 160.02 0)
 			(effects
@@
 			(project "scale-infrared-digitiser"
 				(path "/30c568d4-c8fa-43dd-998e-54c85dfa19bf"
-					(reference "D_photo3")
+					(reference "DPht3")
 					(unit 1)
 				)
@@
 	)
 	(symbol
-		(lib_name "VEMD10940FX01_1")
 		(lib_id "Samacsys:VEMD10940FX01")
 		(at 236.22 165.1 0)
@@
 		(on_board yes)
 		(dnp no)
-		(property "Reference" "D_photo5"
+		(property "Reference" "DPht5"
 			(at 236.728 160.02 0)
 			(effects
@@
 			(project "scale-infrared-digitiser"
 				(path "/30c568d4-c8fa-43dd-998e-54c85dfa19bf"
-					(reference "D_photo5")
+					(reference "DPht5")
 					(unit 1)
 				)
@@
 	)
 	(symbol
-		(lib_name "VEMD10940FX01_1")
 		(lib_id "Samacsys:VEMD10940FX01")
 		(at 67.31 165.1 0)
@@
 		(on_board yes)
 		(dnp no)
-		(property "Reference" "D_photo1"
+		(property "Reference" "DPht1"
 			(at 67.818 160.02 0)
 			(effects
@@
 			(project "scale-infrared-digitiser"
 				(path "/30c568d4-c8fa-43dd-998e-54c85dfa19bf"
-					(reference "D_photo1")
+					(reference "DPht1")
 					(unit 1)
 				)
@@
 	)
 	(symbol
-		(lib_name "VEMD10940FX01_1")
 		(lib_id "Samacsys:VEMD10940FX01")
 		(at 128.27 165.1 0)
@@
 		(on_board yes)
 		(dnp no)
-		(property "Reference" "D_photo2"
+		(property "Reference" "DPht2"
 			(at 128.778 160.02 0)
 			(effects
@@
 			(project "scale-infrared-digitiser"
 				(path "/30c568d4-c8fa-43dd-998e-54c85dfa19bf"
-					(reference "D_photo2")
+					(reference "DPht2")
 					(unit 1)
 				)
@@
 	)
 	(symbol
-		(lib_name "VEMD10940FX01_1")
 		(lib_id "Samacsys:VEMD10940FX01")
 		(at 107.95 224.79 0)
@@
 		(on_board yes)
 		(dnp no)
-		(property "Reference" "D_photo11"
+		(property "Reference" "DPht11"
 			(at 108.458 219.71 0)
 			(effects
@@
 			(project "scale-infrared-digitiser"
 				(path "/30c568d4-c8fa-43dd-998e-54c85dfa19bf"
-					(reference "D_photo11")
+					(reference "DPht11")
 					(unit 1)
 				)
@@
 	)
 	(symbol
-		(lib_name "VSMB10940_1")
 		(lib_id "Samacsys:VSMB10940")
 		(at 116.84 39.37 0)
@@
 	)
 	(symbol
-		(lib_name "VEMD10940FX01_1")
 		(lib_id "Samacsys:VEMD10940FX01")
 		(at 67.31 224.79 0)
@@
 		(on_board yes)
 		(dnp no)
-		(property "Reference" "D_photo9"
+		(property "Reference" "DPht9"
 			(at 67.818 219.71 0)
 			(effects
@@
 			(project "scale-infrared-digitiser"
 				(path "/30c568d4-c8fa-43dd-998e-54c85dfa19bf"
-					(reference "D_photo9")
+					(reference "DPht9")
 					(unit 1)
 				)
