File: scale-infrared-digitiser-receiver.kicad_sch (KiCad schematic)
At the start: 60 parts, among them IC0 LM324PT, IC1 LM324PT, IC2 LM324PT, IC3 LM324PT, J1 Conn_02x04_RECV

Commit message: reworking to exclude amplifiers - may need to rollback
Parts:
- removed C1, C10, C11, C12, C15, C16, C17, C18, C21, C22, C23, C24, C3, C4, C5, C9: 5.1p, Capacitor_SMD:C_0603_1608Metric, symbol Device:C_Small
- removed C14, C2, C20, C7, C8: 1u, Capacitor_SMD:C_0603_1608Metric, symbol Device:C_Small
- removed IC0, IC1, IC2, IC3: LM324PT, Samacsys:SOP65P640X120-14N, symbol Samacsys:LM324PT
- removed J1: Conn_02x04_RECV, Connector_PinHeader_2.54mm:PinHeader_2x04_P2.54mm_Vertical, symbol Connector_Generic:Conn_02x04_Top_Bottom
- removed R17, R20, R21, R22, R23, R24, R25, R26, R27, R28, R29, R30, R31, R32, R33, R34: 750k, Resistor_SMD:R_0603_1608Metric, symbol Device:R_Small
- removed R18: 115k, Resistor_SMD:R_0603_1608Metric, symbol Device:R_Small
- removed R19: 3.57k, Resistor_SMD:R_0603_1608Metric, symbol Device:R_Small
- added J0: Conn_01x16, symbol Connector_Generic:Conn_01x16
Connections:
- net GND: now also J0.1 (Pin_1)
- net PHT_DAT_0: now also DPht0.1 (K), J0.16 (Pin_16)
- net PHT_DAT_1: now also DPht1.1 (K), J0.15 (Pin_15)
- net PHT_DAT_10: now also DPht10.1 (K), J0.6 (Pin_6)
- net PHT_DAT_11: now also DPht11.1 (K), J0.5 (Pin_5)
- net PHT_DAT_12: now also DPht12.1 (K), J0.4 (Pin_4)
- net PHT_DAT_13: now also DPht13.1 (K), J0.3 (Pin_3)
- net PHT_DAT_14: now also DPht14.1 (K), J0.2 (Pin_2)
- net PHT_DAT_15: now also DPht15.1 (K)
- net PHT_DAT_2: now also DPht2.1 (K), J0.14 (Pin_14)
- net PHT_DAT_3: now also DPht3.1 (K), J0.13 (Pin_13)
- net PHT_DAT_4: now also DPht4.1 (K), J0.12 (Pin_12)
- net PHT_DAT_5: now also DPht5.1 (K), J0.11 (Pin_11)
- net PHT_DAT_6: now also DPht6.1 (K), J0.10 (Pin_10)
- net PHT_DAT_7: now also DPht7.1 (K), J0.9 (Pin_9)
- net PHT_DAT_8: now also DPht8.1 (K), J0.8 (Pin_8)
- net PHT_DAT_9: now also DPht9.1 (K), J0.7 (Pin_7)
Other:
- moved on the sheet: DPht0, DPht1, DPht10, DPht11, DPht12, DPht13, DPht14, DPht15, DPht2, DPht3, DPht4, DPht5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
