File: scale-infrared-digitiser-receiver.kicad_sch (KiCad schematic)
At the start: 111 parts, among them IC0 LM324PT, IC1 LM324PT, IC2 LM324PT, IC3 LM324PT, IC4 74HC4067PW,118, IC5 74HC4067PW,118, J0 Conn_02x04_TRNS, J1 Conn_02x04_RECV, Q1 T2N7002AK, Q10 T2N7002AK, Q11 T2N7002AK, Q12 T2N7002AK, Q13 T2N7002AK, Q14 T2N7002AK, Q15 T2N7002AK, Q16 T2N7002AK, Q2 T2N7002AK, Q3 T2N7002AK, Q4 T2N7002AK, Q5 T2N7002AK, Q6 T2N7002AK, Q7 T2N7002AK, Q8 T2N7002AK, Q9 T2N7002AK

Commit message: working on updated receiver pcb
Parts:
- removed IC4, IC5: 74HC4067PW,118, Samacsys:SOP65P640X110-24N, symbol Samacsys:74HC4067PW,118
- removed J0: Conn_02x04_TRNS, Connector_PinHeader_2.54mm:PinHeader_2x04_P2.54mm_Vertical, symbol Connector_Generic:Conn_02x04_Top_Bottom
- removed J1: Conn_02x04_RECV, Connector_PinHeader_2.54mm:PinHeader_2x04_P2.54mm_Vertical, symbol Connector_Generic:Conn_02x04_Top_Bottom
- removed LED0, LED1, LED10, LED11, LED12, LED13, LED14, LED15, LED2, LED3, LED4, LED5, LED6, LED7, LED8, LED9: VSMB10940, Samacsys:VSMB10940, symbol Samacsys:VSMB10940
- removed Q1, Q10, Q11, Q12, Q13, Q14, Q15, Q16, Q2, Q3, Q4, Q5, Q6, Q7, Q8, Q9: T2N7002AK, Package_TO_SOT_SMD:SOT-23, symbol Transistor_FET:T2N7002AK
- removed R1, R10, R11, R12, R13, R14, R15, R16, R2, R3, R4, R5, R6, R7, R8, R9: 200R, Resistor_SMD:R_0603_1608Metric, symbol Device:R_Small
- added J0: Conn_01x18, symbol Connector_Generic:Conn_01x18
Connections:
- net PHT_DAT_0_R is gone; now on net PHT_DAT_0: C9.2, IC0.1 (OUTPUT_1), R23.1
- net PHT_DAT_10_R is gone; now on net PHT_DAT_10: C22.1, IC3.7 (OUTPUT_2), R32.2
- net PHT_DAT_11_R is gone; now on net PHT_DAT_11: C21.2, IC3.1 (OUTPUT_1), R31.1
- net PHT_DAT_12_R is gone; now on net PHT_DAT_12: C1.2, IC2.1 (OUTPUT_1), R17.1
- net PHT_DAT_13_R is gone; now on net PHT_DAT_13: C4.1, IC2.7 (OUTPUT_2), R21.2
- net PHT_DAT_14_R is gone; now on net PHT_DAT_14: C5.2, IC2.8 (OUTPUT_3), R22.1
- net PHT_DAT_15_R is gone; now on net PHT_DAT_15: C3.1, IC2.14 (OUTPUT_4), R20.2
- net PHT_DAT_1_R is gone; now on net PHT_DAT_1: C10.1, IC0.7 (OUTPUT_2), R24.2
- net PHT_DAT_2_R is gone; now on net PHT_DAT_2: C11.2, IC0.8 (OUTPUT_3), R25.1
- net PHT_DAT_3_R is gone; now on net PHT_DAT_3: C12.1, IC0.14 (OUTPUT_4), R26.2
- net PHT_DAT_4_R is gone; now on net PHT_DAT_4: C15.2, IC1.1 (OUTPUT_1), R27.1
- net PHT_DAT_5_R is gone; now on net PHT_DAT_5: C16.1, IC1.7 (OUTPUT_2), R28.2
- net PHT_DAT_6_R is gone; now on net PHT_DAT_6: C17.2, IC1.8 (OUTPUT_3), R29.1
- net PHT_DAT_7_R is gone; now on net PHT_DAT_7: C18.1, IC1.14 (OUTPUT_4), R30.2
- net PHT_DAT_8_R is gone; now on net PHT_DAT_8: C24.1, IC3.14 (OUTPUT_4), R34.2
- net PHT_DAT_9_R is gone; now on net PHT_DAT_9: C23.2, IC3.8 (OUTPUT_3), R33.1
- net 3V3_RECV: now also J0.1 (Pin_1)
- net GND: now also J0.18 (Pin_18)
- net PHT_DAT_0: now also J0.2 (Pin_2); no longer C9.1, DPht1.1 (K), IC0.2 (INVERTING_INPUT_1), R23.2
- net PHT_DAT_1: now also J0.3 (Pin_3); no longer C10.2, DPht0.1 (K), IC0.6 (INVERTING_INPUT_2), R24.1
- net PHT_DAT_10: now also J0.12 (Pin_12); no longer C22.2, DPht12.1 (K), IC3.6 (INVERTING_INPUT_2), R32.1
- net PHT_DAT_11: now also J0.13 (Pin_13); no longer C21.1, DPht13.1 (K), IC3.2 (INVERTING_INPUT_1), R31.2
- net PHT_DAT_12: now also J0.14 (Pin_14); no longer C1.1, DPht9.1 (K), IC2.2 (INVERTING_INPUT_1), R17.2
- net PHT_DAT_13: now also J0.15 (Pin_15); no longer C4.2, DPht8.1 (K), IC2.6 (INVERTING_INPUT_2), R21.1
- net PHT_DAT_14: now also J0.16 (Pin_16); no longer C5.1, DPht11.1 (K), IC2.9 (INVERTING_INPUT_3), R22.2
- net PHT_DAT_15: now also J0.17 (Pin_17); no longer C3.2, DPht10.1 (K), IC2.13 (INVERTING_INPUT_4), R20.1
- net PHT_DAT_2: now also J0.4 (Pin_4); no longer C11.1, DPht3.1 (K), IC0.9 (INVERTING_INPUT_3), R25.2
- net PHT_DAT_3: now also J0.5 (Pin_5); no longer C12.2, DPht2.1 (K), IC0.13 (INVERTING_INPUT_4), R26.1
- net PHT_DAT_4: now also J0.6 (Pin_6); no longer C15.1, DPht5.1 (K), IC1.2 (INVERTING_INPUT_1), R27.2
- net PHT_DAT_5: now also J0.7 (Pin_7); no longer C16.2, DPht4.1 (K), IC1.6 (INVERTING_INPUT_2), R28.1
- net PHT_DAT_6: now also J0.8 (Pin_8); no longer C17.1, DPht7.1 (K), IC1.9 (INVERTING_INPUT_3), R29.2
- net PHT_DAT_7: now also J0.9 (Pin_9); no longer C18.2, DPht6.1 (K), IC1.13 (INVERTING_INPUT_4), R30.1
- net PHT_DAT_8: now also J0.10 (Pin_10); no longer C24.2, DPht14.1 (K), IC3.13 (INVERTING_INPUT_4), R34.1
- net PHT_DAT_9: now also J0.11 (Pin_11); no longer C23.1, DPht15.1 (K), IC3.9 (INVERTING_INPUT_3), R33.2
- new net: C18.2, DPht6.1 (K), IC1.13 (INVERTING_INPUT_4), R30.1
- new net: C3.2, DPht10.1 (K), IC2.13 (INVERTING_INPUT_4), R20.1
- new net: C16.2, DPht4.1 (K), IC1.6 (INVERTING_INPUT_2), R28.1
- new net: C17.1, DPht7.1 (K), IC1.9 (INVERTING_INPUT_3), R29.2
- new net: C24.2, DPht14.1 (K), IC3.13 (INVERTING_INPUT_4), R34.1
- new net: C15.1, DPht5.1 (K), IC1.2 (INVERTING_INPUT_1), R27.2
- new net: C4.2, DPht8.1 (K), IC2.6 (INVERTING_INPUT_2), R21.1
- new net: C11.1, DPht3.1 (K), IC0.9 (INVERTING_INPUT_3), R25.2
- new net: C9.1, DPht1.1 (K), IC0.2 (INVERTING_INPUT_1), R23.2
- new net: C10.2, DPht0.1 (K), IC0.6 (INVERTING_INPUT_2), R24.1
- new net: C12.2, DPht2.1 (K), IC0.13 (INVERTING_INPUT_4), R26.1
- new net: C23.1, DPht15.1 (K), IC3.9 (INVERTING_INPUT_3), R33.2
- new net: C5.1, DPht11.1 (K), IC2.9 (INVERTING_INPUT_3), R22.2
- new net: C22.2, DPht12.1 (K), IC3.6 (INVERTING_INPUT_2), R32.1
- new net: C21.1, DPht13.1 (K), IC3.2 (INVERTING_INPUT_1), R31.2
- new net: C1.1, DPht9.1 (K), IC2.2 (INVERTING_INPUT_1), R17.2
- no-connect marks 32 -> 16
Other:
- note removed: "Transmitter array"
